File: PEEKbot_APS.kicad_pcb (KiCad board)
At the start: 2 copper layers, 90 parts, among them J1 Conn_01x05, J2 Conn_01x05, J3 Conn_01x02, J4 Conn_01x03_Pin, J5 Conn_01x03_Pin, J6 Conn_01x01_Pin, J7 Conn_01x01_Pin, Q1 2N7002, Q2 2N7002, Q3 2N7002, Q4 2N7002, SW1 SW_DIP_x04, SW2 RotaryEncoder, SW3 RotaryEncoder, U1 TLV76118, U2 TPS62933, U3 TMP300, U4 STM32G071CBTx, U5 SN65HVD72DRBR, U6 DRV10974RUMR, U7 DRV10974RUMR

Commit message: Add files via upload
1st iteration finalized. The board has been tested and partially debugged. Comments can be found in the txt file.
Parts:
- removed C21, C22: 1uF, Capacitor_SMD:C_0603_1608Metric_Pad1.08x0.95mm_HandSolder
- removed J6, J7: Conn_01x01_Pin, Connector_Wire:SolderWirePad_1x01_SMD_1x2mm
- removed LD1: D_Laser, Connector_JST:JST_EH_S2B-EH_1x02_P2.50mm_Horizontal
- removed R26, R28, R29, R30, R38, R39: 10k, Resistor_SMD:R_0603_1608Metric_Pad0.98x0.95mm_HandSolder
- removed R27, R35, R36, R37: 0, Resistor_SMD:R_0603_1608Metric_Pad0.98x0.95mm_HandSolder
- removed R31, R33: 120k, Resistor_SMD:R_0603_1608Metric_Pad0.98x0.95mm_HandSolder
- removed R32, R34: 36k, Resistor_SMD:R_0402_1005Metric_Pad0.72x0.64mm_HandSolder
- removed S2, S3: D2FS, Connector_PinHeader_1.27mm:PinHeader_1x03_P1.27mm_Vertical
- removed SW2, SW3: RotaryEncoder, Connector_PinHeader_1.27mm:PinHeader_1x03_P1.27mm_Vertical
- added H1: MountingHole_Pad, Connector_Wire:SolderWire-0.5sqmm_1x01_D0.9mm_OD2.3mm, F.Cu at (18.1, 180.6)
- added H2: MountingHole_Pad, Connector_Wire:SolderWire-0.5sqmm_1x01_D0.9mm_OD2.3mm, F.Cu at (18.1, 174.0)
- added H3: MountingHole_Pad, Connector_Wire:SolderWire-0.5sqmm_1x01_D0.9mm_OD2.3mm, F.Cu at (18.1, 177.3)
- added H4: MountingHole_Pad, Connector_Wire:SolderWire-0.5sqmm_1x01_D0.9mm_OD2.3mm, F.Cu at (18.1, 170.7)
- added H5: MountingHole_Pad, Connector_Wire:SolderWire-0.5sqmm_1x01_D0.9mm_OD2.3mm, F.Cu at (18.1, 187.2)
- added H6: MountingHole_Pad, Connector_Wire:SolderWire-0.5sqmm_1x01_D0.9mm_OD2.3mm, F.Cu at (18.1, 183.9)
- added JP3: SolderJumper_2_Open, Jumper:SolderJumper-2_P1.3mm_Open_RoundedPad1.0x1.5mm, F.Cu at (27.4, 174.5)
- added JP4: SolderJumper_2_Open, Jumper:SolderJumper-2_P1.3mm_Open_RoundedPad1.0x1.5mm, F.Cu at (27.4, 177.0)
- added JP5: SolderJumper_2_Open, Jumper:SolderJumper-2_P1.3mm_Open_RoundedPad1.0x1.5mm, F.Cu at (26.9, 185.9)
- added L2: 6.3uH, Inductor_SMD:L_Bourns_SRN6045TA, F.Cu at (31.7, 156.7)
- added TP1: TestPoint_Probe, TestPoint:TestPoint_Pad_D1.5mm, B.Cu at (25.7, 155.3)
- added TP2: TestPoint_Probe, TestPoint:TestPoint_Pad_D1.5mm, F.Cu at (37.0, 168.7)
- added TP3: TestPoint_Probe, TestPoint:TestPoint_Pad_D1.5mm, F.Cu at (53.0, 145.8)
- added TP4: TestPoint_Probe, TestPoint:TestPoint_Pad_D1.5mm, F.Cu at (52.1, 143.0)
- added U8: DRV8220DSGR-8p, Package_SON:WSON-8-1EP_2x2mm_P0.5mm_EP0.9x1.6mm_ThermalVias, B.Cu at (22.8, 184.6)
- added VR1: TC33X-2-303E, Potentiometer_SMD:Potentiometer_Bourns_TC33X_Vertical, F.Cu at (22.3, 171.2)
- C1, C3: value 100nF -> 15pF; footprint Capacitor_SMD:C_0603_1608Metric_Pad1.08x0.95mm_HandSolder -> Capacitor_SMD:C_0402_1005Metric_Pad0.74x0.62mm_HandSolder; moved to B.Cu
- C11: value 22uF -> 0.47uF; footprint Capacitor_SMD:C_0805_2012Metric_Pad1.18x1.45mm_HandSolder -> Capacitor_SMD:C_0603_1608Metric_Pad1.08x0.95mm_HandSolder
- C12: value 4.7uF -> 22uF; moved to B.Cu
- C13: value 4.7uF -> 100nF; footprint Capacitor_SMD:C_0805_2012Metric_Pad1.18x1.45mm_HandSolder -> Capacitor_SMD:C_0603_1608Metric_Pad1.08x0.95mm_HandSolder
- C14, C16, C19, C5, C6, R14, R17, R21: moved to B.Cu
- C15, C17: value 100nF -> 22uF; footprint Capacitor_SMD:C_0603_1608Metric_Pad1.08x0.95mm_HandSolder -> Capacitor_SMD:C_0805_2012Metric_Pad1.18x1.45mm_HandSolder; moved to B.Cu
- C18, C20: value 100nF -> 22uF; footprint Capacitor_SMD:C_0603_1608Metric_Pad1.08x0.95mm_HandSolder -> Capacitor_SMD:C_0805_2012Metric_Pad1.18x1.45mm_HandSolder
- C2: value 15pF -> 100nF; footprint Capacitor_SMD:C_0402_1005Metric_Pad0.74x0.62mm_HandSolder -> Capacitor_SMD:C_0603_1608Metric_Pad1.08x0.95mm_HandSolder
- C4: value 15pF -> 100nF; footprint Capacitor_SMD:C_0402_1005Metric_Pad0.74x0.62mm_HandSolder -> Capacitor_SMD:C_0603_1608Metric_Pad1.08x0.95mm_HandSolder; moved to B.Cu
- C7: value 100nF -> 4.7uF; moved to B.Cu
- C9: value 22uF -> 4.7uF; footprint Capacitor_SMD:C_0805_2012Metric_Pad1.18x1.45mm_HandSolder -> Capacitor_SMD:C_0603_1608Metric_Pad1.08x0.95mm_HandSolder; moved to B.Cu
- ESD1: footprint Package_TO_SOT_SMD:SOT-23-3 -> Package_TO_SOT_SMD:SOT-23_Handsoldering; moved to B.Cu
- F1: footprint Fuse:Fuse_0603_1608Metric_Pad1.05x0.95mm_HandSolder -> Capacitor_SMD:C_0805_2012Metric_Pad1.18x1.45mm_HandSolder
- J1: value Conn_01x05 -> Conn_01x02; footprint Connector_PinHeader_1.27mm:PinHeader_1x05_P1.27mm_Horizontal -> Connector_PinHeader_2.54mm:PinHeader_1x02_P2.54mm_Vertical
- J2: footprint Connector_PinHeader_1.27mm:PinHeader_1x05_P1.27mm_Horizontal -> Connector_PinHeader_2.54mm:PinHeader_1x05_P2.54mm_Vertical
- J3: value Conn_01x02 -> 0705430109; footprint Connector_JST:JST_EH_S2B-EH_1x02_P2.50mm_Horizontal -> Connector_PinHeader_2.54mm:PinHeader_1x05_P2.54mm_Vertical
- J4: value Conn_01x03_Pin -> 0705430109; footprint Connector_PinHeader_1.27mm:PinHeader_1x03_P1.27mm_Vertical -> Connector_PinHeader_2.54mm:PinHeader_1x05_P2.54mm_Vertical
- J5: value Conn_01x03_Pin -> Conn_01x02; footprint Connector_PinHeader_1.27mm:PinHeader_1x03_P1.27mm_Vertical -> Connector_PinHeader_2.54mm:PinHeader_1x02_P2.54mm_Vertical
- LSE1: value JTX310 - Jauch -> ECS-.327-12.5-16-TR3; footprint Crystal:Crystal_SMD_3215-2Pin_3.2x1.5mm -> Crystal:Crystal_SMD_MicroCrystal_CM9V-T1A-2Pin_1.6x1.0mm_HandSoldering; moved to B.Cu
- Q1, Q2: value 2N7002 -> 2N7002LT3G
- Q3, Q4: value 2N7002 -> 2N7002LT3G; moved to B.Cu
- R1, R10: value 36k -> 10k; footprint Resistor_SMD:R_0402_1005Metric_Pad0.72x0.64mm_HandSolder -> Resistor_SMD:R_0603_1608Metric_Pad0.98x0.95mm_HandSolder; moved to B.Cu
- R11: value 10k -> 31.3k
- R12: value 0 -> 10k
- R13: value 0 -> Heater; footprint Resistor_SMD:R_0603_1608Metric_Pad0.98x0.95mm_HandSolder -> LED_SMD:LED_0603_1608Metric_Pad1.05x0.95mm_HandSolder
- R19: value R_Photo -> 10k; footprint Connector_JST:JST_EH_S2B-EH_1x02_P2.50mm_Horizontal -> Resistor_SMD:R_0603_1608Metric_Pad0.98x0.95mm_HandSolder; moved to B.Cu
- R2: value 0 -> 10k; footprint Jumper:SolderJumper-2_P1.3mm_Open_TrianglePad1.0x1.5mm -> Resistor_SMD:R_0603_1608Metric_Pad0.98x0.95mm_HandSolder; moved to B.Cu
- R20: value 10k -> 31.3k; moved to B.Cu
- R22, R23, R24: value 10k -> 0; moved to B.Cu
- R25: value 0 -> 50
- R3, R4: value 120k -> 10; moved to B.Cu
- R5: value 1k -> 10k; footprint Resistor_SMD:R_0402_1005Metric_Pad0.72x0.64mm_HandSolder -> Resistor_SMD:R_0603_1608Metric_Pad0.98x0.95mm_HandSolder
- R6: value Heater -> 10k; footprint Jumper:SolderJumper-2_P1.3mm_Open_TrianglePad1.0x1.5mm -> Resistor_SMD:R_0603_1608Metric_Pad0.98x0.95mm_HandSolder
- R7: value 0 -> 10k; footprint Jumper:SolderJumper-2_P1.3mm_Open_TrianglePad1.0x1.5mm -> Resistor_SMD:R_0603_1608Metric_Pad0.98x0.95mm_HandSolder
- R8: value 120k -> 10k
- R9: value 16k -> 30k; footprint Resistor_SMD:R_0402_1005Metric_Pad0.72x0.64mm_HandSolder -> Resistor_SMD:R_0603_1608Metric_Pad0.98x0.95mm_HandSolder
- SW1: footprint Button_Switch_SMD:SW_DIP_SPSTx04_Slide_6.7x11.72mm_W8.61mm_P2.54mm_LowProfile -> Button_Switch_SMD:SW_DIP_SPSTx04_Slide_KingTek_DSHP04TS_W7.62mm_P1.27mm
- U1: value TLV76118 -> SN65HVD72DRBR; footprint Package_TO_SOT_SMD:SOT-223 -> Package_SO:SOIC-8-1EP_3.9x4.9mm_P1.27mm_EP2.29x3mm_ThermalVias; moved to B.Cu
- U2: value TPS62933 -> DRV5011; footprint Package_TO_SOT_SMD:SOT-583-8 -> Package_TO_SOT_THT:TO-92Flat
- U3: value TMP300 -> STM32G071CBT6; footprint Package_TO_SOT_SMD:SOT-23-6_Handsoldering -> Package_QFP:LQFP-48_7x7mm_P0.5mm; moved to B.Cu
- U4: value STM32G071CBTx -> DRV5011; footprint Package_QFP:LQFP-48_7x7mm_P0.5mm -> Package_TO_SOT_THT:TO-92Flat
- U5: value SN65HVD72DRBR -> TMP300; footprint Library:VSSOP-8_3.0x3.0mm_PO0.65mm-EPAD -> Package_TO_SOT_SMD:SOT-363_SC-70-6
- U6: value DRV10974RUMR -> DRV8428; footprint Package_DFN_QFN:WQFN-16-1EP_4x4mm_P0.5mm_EP2.6x2.6mm_ThermalVias -> Package_DFN_QFN:WQFN-16-1EP_3x3mm_P0.5mm_EP1.68x1.68mm_ThermalVias; moved to B.Cu
- U7: value DRV10974RUMR -> TPS62933; footprint Package_DFN_QFN:WQFN-16-1EP_4x4mm_P0.5mm_EP2.6x2.6mm_ThermalVias -> Package_TO_SOT_SMD:SOT-583-8; moved to B.Cu
- moved U2 282.5 mm to (24.8, 192.5), turned to 15 degrees
- moved C10 265.5 mm to (41.6, 181.3), turned to 45 degrees
- moved C11 258.1 mm to (26.1, 172.5), turned to 180 degrees
- moved R11 256.3 mm to (37.5, 172.4), turned to 180 degrees
- moved L1 254.2 mm to (33.6, 164.5), turned to 45 degrees
- moved R10 254.2 mm to (39.9, 173.6), turned to -90 degrees
- moved C6 245.2 mm to (46.7, 157.5), turned to 0 degrees
- moved R7 236.7 mm to (38.8, 147.1), turned to -60 degrees
- moved C9 236.0 mm to (44.3, 156.2), turned to 90 degrees
- moved C5 217.1 mm to (46.7, 155.9), turned to 0 degrees
- moved R14 213.8 mm to (33.6, 172.7)
- moved C1 213.5 mm to (40.8, 159.1), turned to 180 degrees
- moved R2 212.3 mm to (43.0, 142.0), turned to 30 degrees
- moved C18 210.2 mm to (22.8, 186.8)
- moved U1 209.2 mm to (43.1, 146.1), turned to -150 degrees
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Connections:
- C1 pad 1: Vin -> LSE_IN
- C10 pad 1: Net-(U2-SS) -> +3V3
- C11 pad 1: Net-(C11-Pad1) -> GND
- C11 pad 2: GND -> STEP_DVDD
- C12 pad 1: +3V3 -> +12V
- C13 pad 1: +3V3 -> EN
- C14 pad 1: NRST -> Net-(U7-SW)
- C14 pad 2: GND -> Net-(U7-BST)
- C15 pad 1: VREF+ -> Net-(C15-Pad1)
- C16 pad 1: END_LON -> Net-(U7-SS)
- C17 pad 1: END_LAT -> Net-(C15-Pad1)
- C18 pad 1: +3V3 -> GND
- C18 pad 2: GND -> +12V
- C19 pad 1: VCC -> GND
- C19 pad 2: Net-(U6-VCP) -> +12V
- C2 pad 1: LSE_IN -> NRST
- C20 pad 1: VCC -> Net-(C20-Pad1)
- C20 pad 2: Net-(U7-VCP) -> GND
- C3 pad 1: Net-(U3-TSET) -> LSE_OUT
- C4 pad 1: LSE_OUT -> +3V3
- C5 pad 1: Net-(C5-Pad1) -> +3V3
- C6 pad 1: Net-(U2-SW) -> +3V3
- C6 pad 2: Net-(U2-BST) -> GND
- C9 pad 1: Net-(C11-Pad1) -> +3V3
- F1 pad 1: Net-(J6-Pin_1) -> VCC
- F1 pad 2: VCC -> +12V
- J1 pad 1: GND -> OUT_B
- J1 pad 2: SWDCLK -> OUT_A
- J2 pad 1: +3V3 -> GND
- J2 pad 2: CLK-PROBE -> SWDCLK
- J2 pad 3: UART1_TxD -> SWDIO
- J2 pad 4: UART1_RxD -> NRST
- J2 pad 5: GND -> +3V3
- J3 pad 1: OUT_B -> ENC_B_AZM
- J3 pad 2: OUT_A -> +3V3
- J4 pad 1: W_LAT -> ENC_B_ALT
- J4 pad 2: V_LAT -> +3V3
- J4 pad 3: U_LAT -> ENC_A_ALT
- J5 pad 1: W_LON -> VCC
- J5 pad 2: V_LON -> GND
- L1 pad 1: Net-(U2-SW) -> Net-(U7-SW)
- L1 pad 2: Net-(C11-Pad1) -> Net-(C15-Pad1)
- Q2 pad 3: EN -> Net-(Q1-G)
- Q3 pad 1: Net-(Q2-G) -> Net-(Q1-G)
- Q3 pad 3: Net-(Q1-D) -> EN
- Q4 pad 1: LASER -> Net-(Q4-G)
- Q4 pad 3: Net-(LD1-K) -> Net-(Q1-D)
- R1 pad 1: GND -> LPUART_DE
- R1 pad 2: Net-(U3-TSET) -> GND
- R10 pad 1: FB-3.65V -> TEMP
- R10 pad 2: Net-(C11-Pad1) -> GND
- R11 pad 2: FB-3.65V -> Net-(U5-TSET)
- R12 pad 1: Net-(LD1-A) -> +12V
- R12 pad 2: +3V3 -> Net-(Q1-G)
- R13 pad 1: +3V3 -> Net-(Q1-D)
- R13 pad 2: VREF+ -> +12V
- R14 pad 1: NRST -> MOFF
- R14 pad 2: +3V3 -> GND
- R15 pad 1: GND -> Net-(Q2-G)
- R15 pad 2: CFG1 -> MOFF
- R16 pad 1: GND -> +12V
- R16 pad 2: CFG2 -> EN
- R17 pad 1: GND -> HEAT
- R17 pad 2: CFG3 -> Net-(Q4-G)
- R18 pad 1: GND -> HEAT
- R18 pad 2: CFG4 -> GND
- R19 pad 1: VREF+ -> EN
- R19 pad 2: PHO_RES -> GND
- R2 pad 2: Net-(C5-Pad1) -> LP_RxD
- R20 pad 1: GND -> FB-3.3V
- R20 pad 2: PHO_RES -> Net-(C15-Pad1)
- R21 pad 1: GND -> FB-3.3V
- R21 pad 2: END_LON -> GND
- R22 pad 1: GND -> +3V3
- R22 pad 2: END_LAT -> Net-(C20-Pad1)
- R23 pad 1: ENC_LAT_A -> +3V3
- R23 pad 2: +3V3 -> Net-(C20-Pad1)
- R24 pad 1: ENC_LAT_B -> +3V3
- R24 pad 2: +3V3 -> Net-(C20-Pad1)
- R25 pad 1: Net-(R25-Pad1) -> OUT_A
- R25 pad 2: GND -> OUT_B
- R3 pad 1: VCC -> OUT_A
- R3 pad 2: Net-(Q2-G) -> Net-(U1-A)
- R4 pad 1: Net-(Q1-G) -> OUT_B
- R4 pad 2: GND -> Net-(U1-B)
- R5 pad 1: Net-(Q1-G) -> CFG1
- R5 pad 2: HEAT -> GND
- R6 pad 1: Net-(Q1-D) -> CFG2
- R6 pad 2: VCC -> GND
- R7 pad 1: Vin -> CFG3
- R7 pad 2: Net-(C11-Pad1) -> GND
- R8 pad 1: VCC -> CFG4
- R8 pad 2: EN -> GND
- R9 pad 1: GND -> Net-(U5-VTEMP)
- R9 pad 2: EN -> TEMP
- SW1 pad 5: CFG4 -> CFG1
- SW1 pad 6: CFG3 -> CFG2
- SW1 pad 7: CFG2 -> CFG3
- SW1 pad 8: CFG1 -> CFG4
- U1 pad 1: GND -> LP_RxD
- U1 pad 2: Net-(C5-Pad1) -> LPUART_DE
- U1 pad 3: Vin -> LPUART_DE
- U1 pad 4: Net-(C5-Pad1) -> LP_TxD
- U2 pad 1: unconnected-(U2-RT-Pad1) -> +3V3
- U2 pad 2: EN -> END_AZM
- U2 pad 3: VCC -> GND
- U3 pad 1: Net-(U3-TSET) -> unconnected-(U3-PC13-Pad1)
- U3 pad 2: GND -> LSE_IN
- U3 pad 3: Net-(Q2-G) -> LSE_OUT
- U3 pad 4: GND -> +3V3
- U3 pad 5: TEMP -> +3V3
- U4 pad 1: unconnected-(U4-PC13-Pad1) -> +3V3
- U4 pad 2: LSE_IN -> END_ALT
- U4 pad 3: LSE_OUT -> GND
- U5 pad 1: LP_RxD -> Net-(U5-TSET)
- U5 pad 3: LPUART_DE -> Net-(Q1-G)
- U5 pad 4: LP_TxD -> GND
- U5 pad 5: GND -> Net-(U5-VTEMP)
- U5 pad 6: Net-(U5-A) -> +12V
- U6 pad 1: FG_LON -> Net-(U6-AOUT1)
- U6 pad 10: V_LON -> STEP_DVDD
- U6 pad 11: W_LON -> STEP_PWM
- U6 pad 12: VCC -> STEP_DIR
- U6 pad 13: Net-(U6-VCP) -> Net-(JP3-B)
- U6 pad 14: GND -> Net-(JP4-B)
- U6 pad 15: Net-(U6-ADV) -> +12V
- U6 pad 16: FR_LON -> GND
- U6 pad 2: PWM_LON -> Net-(U6-AOUT2)
- U6 pad 6: Net-(U6-CS) -> STEP_DVDD
- U6 pad 7: GND -> Net-(U6-VREF)
- U6 pad 8: unconnected-(U6-NC-Pad8) -> STEP_DVDD
- U6 pad 9: U_LON -> GND
- U7 pad 1: FG_LAT -> unconnected-(U7-RT-Pad1)
- U7 pad 2: PWM_LAT -> EN
- U7 pad 3: Net-(U7-V1P8) -> +12V
- U7 pad 4: Net-(U7-RMP) -> GND
- U7 pad 5: GND -> Net-(U7-SW)
- U7 pad 6: Net-(U7-CS) -> Net-(U7-BST)
- U7 pad 7: GND -> Net-(U7-SS)
- U7 pad 8: unconnected-(U7-NC-Pad8) -> FB-3.3V
Routing:
- net GND: track 0.00 -> 114.7 mm, vias 0 -> 51
- net NRST: track 0.00 -> 50.8 mm, vias 0 -> 1
- net CFG4: track 0.00 -> 43.5 mm, vias 0 -> 2
- net +12V: track 0.00 -> 42.5 mm, vias 0 -> 19
- net END_AZM: track 0.00 -> 38.6 mm, vias 0 -> 1
- net CFG1: track 0.00 -> 37.5 mm, vias 0 -> 1
- net STEP_nSLEEP: track 0.00 -> 37.0 mm, vias 0 -> 2
- net BDC_DIR: track 0.00 -> 34.4 mm, vias 0 -> 2
- net CFG2: track 0.00 -> 33.6 mm, vias 0 -> 1
- net LP_RxD: track 0.00 -> 33.3 mm, vias 0 -> 1
- net BDC_PWM: track 0.00 -> 33.2 mm, vias 0 -> 2
- net STEP_DIR: track 0.00 -> 32.8 mm, vias 0 -> 2
- net STEP_PWM: track 0.00 -> 32.5 mm, vias 0 -> 2
- net BDC_nSLEEP: track 0.00 -> 32.0 mm, vias 0 -> 2
- net STEP_FAULT: track 0.00 -> 31.5 mm, vias 0 -> 2
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- added copper zone on B.Cu, net +12V
- added copper zone on In1.Cu, net +12V
- added copper zone on B.Cu, net +3V3
- added copper zone on In1.Cu, net +3V3
- added copper zone on B.Cu, net GND
- added copper zone on F.Cu, net GND
- added copper zone on In2.Cu, net GND
- added copper zone on B.Cu, net Net-(C15-Pad1)
- added copper zone on F.Cu, net Net-(C15-Pad1)
- added copper zone on B.Cu, net Net-(C20-Pad1)
- added copper zone on F.Cu, net Net-(C20-Pad1)
- added copper zone on B.Cu, net Net-(U6-AOUT1)
- added copper zone on B.Cu, net Net-(U8-OUT1)
- added copper zone on B.Cu, net Net-(U8-OUT2)
Other:
- board outline added: 40 x 59.2 mm
- copper layers 2 -> 4
- board text added: "2023/12/04 V1.1"
- board text added: "A1"
- board text added: "A2"
- board text added: "ALT_A"
- board text added: "ALT_B"
- board text added: "ALT_END"
- board text added: "ALT_I"
- board text added: "AZM_A"
- board text added: "AZM_B"
- board text added: "AZM_END"
- board text added: "AZM_I"
- board text added: "B1"
- board text added: "B2"
- board text added: "BDC1"
- board text added: "BDC2"
- board text added: "GND"
- board text added: "NRST"
- board text added: "RxD"
- board text added: "SWDCK"
- board text added: "SWDIO"
- board text added: "TxD"
- board text added: "VCC"
