File: PEEKbot_APS.kicad_sch (KiCad schematic)
At the start: 78 parts, among them J1 Conn_01x02, J2 Conn_01x05, J3 Conn_01x05, Q1 2N7002, Q2 2N7002, Q3 2N7002, Q4 2N7002, SW1 SW_DIP_x04, SW2 RotaryEncoder, SW3 RotaryEncoder, U1 STM32G071CBTx, U2 TMP300, U4 TLV76118, U5 TPS62933, U6 DRV8220DSGR, U7 DRV8220DSGR, U8 SN65HVD72DRBR

Commit message: Add files via upload
H-bridges for BDC motors replaced with simple BLDC motor drivers (speed control only);
Some 0 Ohm resistors replaced with bridge pads;
All footprints assigned to components (Need to be reviewed, some footprints should be smaller);
Started working on the PCB design
Parts:
- removed C18: 100nF, symbol Device:C_Small
- removed SW2, SW3: RotaryEncoder, symbol Device:RotaryEncoder
- removed U6, U7: DRV8220DSGR, WSON8_DSG_TEX, symbol 1.Texas_Instruments:DRV8220DSGR
- added C19, C20: 100nF, Capacitor_SMD:C_0603_1608Metric_Pad1.08x0.95mm_HandSolder, symbol Device:C_Small
- added C21: 1uF, Capacitor_SMD:C_0603_1608Metric_Pad1.08x0.95mm_HandSolder, symbol Device:C_Small
- added J4, J5: Conn_01x03_Pin, Connector_PinHeader_1.27mm:PinHeader_1x03_P1.27mm_Vertical, symbol Connector:Conn_01x03_Pin
- added J6, J7: Conn_01x01_Pin, Connector_Wire:SolderWirePad_1x01_SMD_1x2mm, symbol Connector:Conn_01x01_Pin
- added R31, R33: 120k, Resistor_SMD:R_0603_1608Metric_Pad0.98x0.95mm_HandSolder, symbol Device:R_Small
- added R32, R34: 36k, Resistor_SMD:R_0402_1005Metric_Pad0.72x0.64mm_HandSolder, symbol Device:R_Small
- added R38, R39: 10k, Resistor_SMD:R_0603_1608Metric_Pad0.98x0.95mm_HandSolder, symbol Device:R_Small
- added SW2, SW3: RotaryEncoder, Connector_PinHeader_1.27mm:PinHeader_1x03_P1.27mm_Vertical, symbol Incremental_Encoder:RotaryEncoder
- added U6, U7: DRV10974RUMR, Package_DFN_QFN:WQFN-16-1EP_4x4mm_P0.5mm_EP2.6x2.6mm_ThermalVias, symbol 1.Texas_Instruments:DRV10974RUMR
- C1: renamed from C2; footprint (none) -> Capacitor_SMD:C_0603_1608Metric_Pad1.08x0.95mm_HandSolder
- C10: renamed from C4; footprint (none) -> Capacitor_SMD:C_0603_1608Metric_Pad1.08x0.95mm_HandSolder
- C11: renamed from C6; footprint (none) -> Capacitor_SMD:C_0805_2012Metric_Pad1.18x1.45mm_HandSolder
- C12: renamed from C15; footprint (none) -> Capacitor_SMD:C_0805_2012Metric_Pad1.18x1.45mm_HandSolder
- C13: renamed from C16; footprint (none) -> Capacitor_SMD:C_0805_2012Metric_Pad1.18x1.45mm_HandSolder
- C14: renamed from C17; footprint (none) -> Capacitor_SMD:C_0603_1608Metric_Pad1.08x0.95mm_HandSolder
- C15: renamed from C19; footprint (none) -> Capacitor_SMD:C_0603_1608Metric_Pad1.08x0.95mm_HandSolder
- C16: renamed from C20; footprint (none) -> Capacitor_SMD:C_0603_1608Metric_Pad1.08x0.95mm_HandSolder
- C17: renamed from C21; footprint (none) -> Capacitor_SMD:C_0603_1608Metric_Pad1.08x0.95mm_HandSolder
- C18: renamed from C7; footprint (none) -> Capacitor_SMD:C_0603_1608Metric_Pad1.08x0.95mm_HandSolder
- C2: renamed from C12; footprint (none) -> Capacitor_SMD:C_0402_1005Metric_Pad0.74x0.62mm_HandSolder
- C22: value 100nF -> 1uF; footprint (none) -> Capacitor_SMD:C_0603_1608Metric_Pad1.08x0.95mm_HandSolder
- C3: renamed from C8; footprint (none) -> Capacitor_SMD:C_0603_1608Metric_Pad1.08x0.95mm_HandSolder
- C4: renamed from C11; footprint (none) -> Capacitor_SMD:C_0402_1005Metric_Pad0.74x0.62mm_HandSolder
- C5: renamed from C1; footprint (none) -> Capacitor_SMD:C_0603_1608Metric_Pad1.08x0.95mm_HandSolder
- C6: renamed from C3; footprint (none) -> Capacitor_SMD:C_0603_1608Metric_Pad1.08x0.95mm_HandSolder
- C7: renamed from C13; footprint (none) -> Capacitor_SMD:C_0603_1608Metric_Pad1.08x0.95mm_HandSolder
- C8: renamed from C14; footprint (none) -> Capacitor_SMD:C_0603_1608Metric_Pad1.08x0.95mm_HandSolder
- C9: renamed from C5; footprint (none) -> Capacitor_SMD:C_0805_2012Metric_Pad1.18x1.45mm_HandSolder
- ESD1, Q4: footprint Package_TO_SOT_SMD:SOT-23 -> Package_TO_SOT_SMD:SOT-23-3
- F1: footprint (none) -> Fuse:Fuse_0603_1608Metric_Pad1.05x0.95mm_HandSolder
- J1: renamed from J3; footprint (none) -> Connector_PinHeader_1.27mm:PinHeader_1x05_P1.27mm_Horizontal
- J2: footprint (none) -> Connector_PinHeader_1.27mm:PinHeader_1x05_P1.27mm_Horizontal
- J3: renamed from J1; footprint (none) -> Connector_JST:JST_EH_S2B-EH_1x02_P2.50mm_Horizontal
- L1: footprint (none) -> Inductor_SMD:L_Bourns_SRN6045TA
- LD1: footprint (none) -> Connector_JST:JST_EH_S2B-EH_1x02_P2.50mm_Horizontal
- LSE1: renamed from LSE; footprint (none) -> Crystal:Crystal_SMD_3215-2Pin_3.2x1.5mm
- Q1: renamed from Q3; footprint Package_TO_SOT_SMD:SOT-23 -> Package_TO_SOT_SMD:SOT-23-3
- Q2: renamed from Q1; footprint Package_TO_SOT_SMD:SOT-23 -> Package_TO_SOT_SMD:SOT-23-3
- Q3: renamed from Q2; footprint Package_TO_SOT_SMD:SOT-23 -> Package_TO_SOT_SMD:SOT-23-3
- R1: renamed from R9; footprint (none) -> Resistor_SMD:R_0402_1005Metric_Pad0.72x0.64mm_HandSolder
- R10: renamed from R3; footprint (none) -> Resistor_SMD:R_0402_1005Metric_Pad0.72x0.64mm_HandSolder
- R11: renamed from R4; footprint (none) -> Resistor_SMD:R_0603_1608Metric_Pad0.98x0.95mm_HandSolder
- R12: renamed from R36; footprint (none) -> Resistor_SMD:R_0603_1608Metric_Pad0.98x0.95mm_HandSolder
- R13: renamed from R29; footprint (none) -> Resistor_SMD:R_0603_1608Metric_Pad0.98x0.95mm_HandSolder
- R14: renamed from R30; footprint (none) -> Resistor_SMD:R_0603_1608Metric_Pad0.98x0.95mm_HandSolder
- R15: renamed from R13; footprint (none) -> Resistor_SMD:R_0603_1608Metric_Pad0.98x0.95mm_HandSolder
- R16: renamed from R14; footprint (none) -> Resistor_SMD:R_0603_1608Metric_Pad0.98x0.95mm_HandSolder
- R17: renamed from R15; footprint (none) -> Resistor_SMD:R_0603_1608Metric_Pad0.98x0.95mm_HandSolder
- R18: renamed from R16; footprint (none) -> Resistor_SMD:R_0603_1608Metric_Pad0.98x0.95mm_HandSolder
- R19: renamed from R34; footprint (none) -> Connector_JST:JST_EH_S2B-EH_1x02_P2.50mm_Horizontal
- R2: renamed from R12; footprint (none) -> Jumper:SolderJumper-2_P1.3mm_Open_TrianglePad1.0x1.5mm
- R20: renamed from R35; footprint (none) -> Resistor_SMD:R_0603_1608Metric_Pad0.98x0.95mm_HandSolder
- R21: renamed from R17; footprint (none) -> Resistor_SMD:R_0603_1608Metric_Pad0.98x0.95mm_HandSolder
- R22: renamed from R37; footprint (none) -> Resistor_SMD:R_0603_1608Metric_Pad0.98x0.95mm_HandSolder
- R23: renamed from R20; footprint (none) -> Resistor_SMD:R_0603_1608Metric_Pad0.98x0.95mm_HandSolder
- R24: renamed from R21; footprint (none) -> Resistor_SMD:R_0603_1608Metric_Pad0.98x0.95mm_HandSolder
- R25: renamed from R19; footprint (none) -> Resistor_SMD:R_0603_1608Metric_Pad0.98x0.95mm_HandSolder
- R26: renamed from R5; footprint (none) -> Resistor_SMD:R_0603_1608Metric_Pad0.98x0.95mm_HandSolder
- R27: renamed from R24; footprint (none) -> Resistor_SMD:R_0603_1608Metric_Pad0.98x0.95mm_HandSolder
- R28: renamed from R22; footprint (none) -> Resistor_SMD:R_0603_1608Metric_Pad0.98x0.95mm_HandSolder
- R29: renamed from R23; footprint (none) -> Resistor_SMD:R_0603_1608Metric_Pad0.98x0.95mm_HandSolder
- R3: renamed from R31; footprint (none) -> Resistor_SMD:R_0603_1608Metric_Pad0.98x0.95mm_HandSolder
- R30: renamed from R8; footprint (none) -> Resistor_SMD:R_0603_1608Metric_Pad0.98x0.95mm_HandSolder
- R35: renamed from R6; footprint (none) -> Resistor_SMD:R_0603_1608Metric_Pad0.98x0.95mm_HandSolder
- R36: renamed from R7; footprint (none) -> Resistor_SMD:R_0603_1608Metric_Pad0.98x0.95mm_HandSolder
- R37: renamed from R18; footprint (none) -> Resistor_SMD:R_0603_1608Metric_Pad0.98x0.95mm_HandSolder
- R4: renamed from R33; footprint (none) -> Resistor_SMD:R_0603_1608Metric_Pad0.98x0.95mm_HandSolder
- R5: renamed from R32; footprint (none) -> Resistor_SMD:R_0402_1005Metric_Pad0.72x0.64mm_HandSolder
- R6: renamed from R11; footprint (none) -> Jumper:SolderJumper-2_P1.3mm_Open_TrianglePad1.0x1.5mm
- R7: renamed from R10; footprint (none) -> Jumper:SolderJumper-2_P1.3mm_Open_TrianglePad1.0x1.5mm
- R8: renamed from R1; footprint (none) -> Resistor_SMD:R_0603_1608Metric_Pad0.98x0.95mm_HandSolder
- R9: renamed from R2; footprint (none) -> Resistor_SMD:R_0402_1005Metric_Pad0.72x0.64mm_HandSolder
- S1: footprint PTS526SK15SMTR2LFS -> Button_Switch_SMD:SW_SPST_TL3342
- S2: renamed from S4; footprint D2FSFLN -> Connector_PinHeader_1.27mm:PinHeader_1x03_P1.27mm_Vertical
- S3: footprint D2FSFLN -> Connector_PinHeader_1.27mm:PinHeader_1x03_P1.27mm_Vertical
- SW1: footprint (none) -> Button_Switch_SMD:SW_DIP_SPSTx04_Slide_6.7x11.72mm_W8.61mm_P2.54mm_LowProfile
- U1: renamed from U4; footprint SOT_8DCYR_TEX -> Package_TO_SOT_SMD:SOT-223
- U2: renamed from U5; footprint SOT_33DRLR_TEX -> Package_TO_SOT_SMD:SOT-583-8
- U3: renamed from U2; footprint DCK6 -> Package_TO_SOT_SMD:SOT-23-6_Handsoldering
- U5: renamed from U8; footprint DRB8_1P65X2P4_TEX -> Library:VSSOP-8_3.0x3.0mm_PO0.65mm-EPAD
- renumbered U1 to U4
Connections:
- net ENC_LAT_A: now also SW3.1
- net ENC_LAT_B: now also SW3.2
- net ENC_LON_A: now also SW2.1
- net ENC_LON_B: now also SW2.2
- net GND: now also C22.1, S1.2 (COM_2), C21.1, J7.1 (Pin_1), R31.2, R32.1, R33.2, R34.1, R38.2, R39.2, U6.14 (GND), U6.17 (PAD), U6.5 (GND), U6.7 (PGND), U7.14 (GND), U7.17 (PAD), U7.5 (GND), U7.7 (PGND); no longer C22.2, S1.3 (NO_1), S1.4 (NO_2)
- net NRST: no longer S1.2 (COM_2)
- net OUT_A: now also ESD1.1 (A1), J3.2 (Pin_2); no longer ESD1.2 (A2), J3.1 (Pin_1)
- net OUT_B: now also ESD1.2 (A2), J3.1 (Pin_1); no longer ESD1.1 (A1), J3.2 (Pin_2)
- net VCC: now also C19.1, C20.1, U6.12 (VCC), U7.12 (VCC); no longer C22.1
- net at R25.1: now also SW3.3
- net at R27.1: now also SW2.3
- net PWR: no longer names the net of F1.1
- net PWR: now also J6.1 (Pin_1)
- new net: R32.2, U6.4 (RMP)
- new net: R34.2, U7.4 (RMP)
- new net: R39.1, U7.6 (CS)
- new net: R38.1, U6.6 (CS)
- new net: R33.1, U7.15 (ADV)
- new net: C19.2, U6.13 (VCP)
- new net: R31.1, U6.15 (ADV)
- new net: C21.2, U6.3 (V1P8)
- new net: C22.2, U7.3 (V1P8)
- new net: C20.2, U7.13 (VCP)
- new net FG_LAT: U7.1 (FG)
- new net FG_LON: U6.1 (FG)
- new net FR_LAT: U7.16 (FR)
- new net FR_LON: U6.16 (FR)
- new net PWM_LAT: U7.2 (PWM)
- new net PWM_LON: U6.2 (PWM)
- new net U_LAT: J4.3 (Pin_3), U7.9 (U)
- new net U_LON: J5.3 (Pin_3), U6.9 (U)
- new net V_LAT: J4.2 (Pin_2), U7.10 (V)
- new net V_LON: J5.2 (Pin_2), U6.10 (V)
- new net W_LAT: J4.1 (Pin_1), U7.11 (W)
- new net W_LON: J5.1 (Pin_1), U6.11 (W)
- no-connect marks 3 -> 5
Other:
- moved on the sheet: C18, ESD1, J3, R26, R30, R35, R36, R37, U5

Commit message: Add files via upload
1st iteration finalized. The board has been tested and partially debugged. Comments can be found in the txt file.
Parts:
- removed C1, C14, C15, C16, C17, C18, C19, C20: 100nF, Capacitor_SMD:C_0603_1608Metric_Pad1.08x0.95mm_HandSolder, symbol Device:C_Small
- removed C11: 22uF, Capacitor_SMD:C_0805_2012Metric_Pad1.18x1.45mm_HandSolder, symbol Device:C_Small
- removed C12, C13: 4.7uF, Capacitor_SMD:C_0805_2012Metric_Pad1.18x1.45mm_HandSolder, symbol Device:C_Small
- removed C21, C22: 1uF, Capacitor_SMD:C_0603_1608Metric_Pad1.08x0.95mm_HandSolder, symbol Device:C_Small
- removed F1: Fuse, Fuse:Fuse_0603_1608Metric_Pad1.05x0.95mm_HandSolder, symbol Device:Fuse
- removed J2: Conn_01x05, Connector_PinHeader_1.27mm:PinHeader_1x05_P1.27mm_Horizontal, symbol Connector:Conn_01x05_Pin
- removed J3: Conn_01x02, Connector_JST:JST_EH_S2B-EH_1x02_P2.50mm_Horizontal, symbol Connector_Generic:Conn_01x02
- removed J4, J5: Conn_01x03_Pin, Connector_PinHeader_1.27mm:PinHeader_1x03_P1.27mm_Vertical, symbol Connector:Conn_01x03_Pin
- removed J6, J7: Conn_01x01_Pin, Connector_Wire:SolderWirePad_1x01_SMD_1x2mm, symbol Connector:Conn_01x01_Pin
- removed L1: 6.3uH, Inductor_SMD:L_Bourns_SRN6045TA, symbol Device:L_Small
- removed LD1: D_Laser, Connector_JST:JST_EH_S2B-EH_1x02_P2.50mm_Horizontal, symbol Device:D_Laser_1C2A
- removed Q1, Q2, Q3, Q4: 2N7002, Package_TO_SOT_SMD:SOT-23-3, symbol Transistor_FET:2N7002
- removed R10, R32, R34: 36k, Resistor_SMD:R_0402_1005Metric_Pad0.72x0.64mm_HandSolder, symbol Device:R_Small
- removed R11, R14, R15, R16, R17, R18, R20, R21, R22, R23, R24, R26, R28, R29, R30, R38, R39: 10k, Resistor_SMD:R_0603_1608Metric_Pad0.98x0.95mm_HandSolder, symbol Device:R_Small
- removed R12, R13, R27, R35, R36, R37: 0, Resistor_SMD:R_0603_1608Metric_Pad0.98x0.95mm_HandSolder, symbol Device:R_Small
- removed R19: R_Photo, Connector_JST:JST_EH_S2B-EH_1x02_P2.50mm_Horizontal, symbol Device:R_Photo
- removed R31, R33: 120k, Resistor_SMD:R_0603_1608Metric_Pad0.98x0.95mm_HandSolder, symbol Device:R_Small
- removed R6: Heater, Jumper:SolderJumper-2_P1.3mm_Open_TrianglePad1.0x1.5mm, symbol Device:Heater
- removed R9: 16k, Resistor_SMD:R_0402_1005Metric_Pad0.72x0.64mm_HandSolder, symbol Device:R_Small
- removed S2, S3: D2FS, Connector_PinHeader_1.27mm:PinHeader_1x03_P1.27mm_Vertical, symbol My_components:D2FS-FL-N
- removed SW2, SW3: RotaryEncoder, Connector_PinHeader_1.27mm:PinHeader_1x03_P1.27mm_Vertical, symbol Incremental_Encoder:RotaryEncoder
- removed U1: TLV76118, Package_TO_SOT_SMD:SOT-223, symbol 1.Texas_Instrments:TLV76118
- removed U2: TPS62933, Package_TO_SOT_SMD:SOT-583-8, symbol 1.Texas_Instrments:TPS62933
- removed U3: TMP300, Package_TO_SOT_SMD:SOT-23-6_Handsoldering, symbol 1.Texas_Instrments:TMP300
- removed U5: SN65HVD72DRBR, Library:VSSOP-8_3.0x3.0mm_PO0.65mm-EPAD, symbol 1.Texas_Instruments:SN65HVD72DRBR
- removed U6, U7: DRV10974RUMR, Package_DFN_QFN:WQFN-16-1EP_4x4mm_P0.5mm_EP2.6x2.6mm_ThermalVias, symbol 1.Texas_Instruments:DRV10974RUMR
- added C2: 100nF, Capacitor_SMD:C_0603_1608Metric_Pad1.08x0.95mm_HandSolder, symbol Device:C_Small
- added J1: Conn_01x02, Connector_PinHeader_2.54mm:PinHeader_1x02_P2.54mm_Vertical, symbol Connector_Generic:Conn_01x02
- added J3, J4: 0705430109, Connector_PinHeader_2.54mm:PinHeader_1x05_P2.54mm_Vertical, symbol Connector_Generic:Conn_01x05
- added R6: 10k, Resistor_SMD:R_0603_1608Metric_Pad0.98x0.95mm_HandSolder, symbol Device:R_Small
- added TP1, TP3, TP4: TestPoint_Probe, TestPoint:TestPoint_Pad_D1.5mm, symbol Connector:TestPoint_Probe
- added U1: SN65HVD72DRBR, Package_SO:SOIC-8-1EP_3.9x4.9mm_P1.27mm_EP2.29x3mm_ThermalVias, symbol 1.Texas_Instruments:SN65HVD72DRBR
- added U2, U4: DRV5011, Package_TO_SOT_THT:TO-92Flat, symbol 1.Texas_Instrments:DRV5011ADLPG
- C1: renamed from C2; Manufacturer (none) -> Walsin Technology Corporation; Manufacturer Part Number (none) -> 0603N150J500CT; Supplier (none) -> digikey; Supplier P/N  (none) -> 1292-1487-1-ND; Unit Cost (none) -> 0.15; Weblink (none) -> https://www.digikey.ca/en/products/detail/walsin-technology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
- C10, C5, C6, C8: Manufacturer (none) -> Samsung Electro-Mechanics; Manufacturer Part Number (none) -> CL10B104KB8NNNC; Supplier (none) -> digikey; Supplier P/N  (none) -> 1271276-1000-1-ND; Unit Cost (none) -> 0.15; Weblink (none) -> https://www.digikey.ca/en/products/detail/samsung-electro-m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
- C3: value 100nF -> 15pF; footprint Capacitor_SMD:C_0603_1608Metric_Pad1.08x0.95mm_HandSolder -> Capacitor_SMD:C_0402_1005Metric_Pad0.74x0.62mm_HandSolder; Manufacturer (none) -> digikey; Manufacturer Part Number (none) -> 0603N150J500CT; Supplier (none) -> (effects (font (size 1.27 1.27)) (justify left)); Supplier P/N  (none) -> 1292-1487-1-ND; Unit Cost (none) -> ); Weblink (none) -> https://www.digikey.ca/en/products/detail/walsin-technology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
- C4: value 15pF -> 100nF; footprint Capacitor_SMD:C_0402_1005Metric_Pad0.74x0.62mm_HandSolder -> Capacitor_SMD:C_0603_1608Metric_Pad1.08x0.95mm_HandSolder; Manufacturer (none) -> Samsung Electro-Mechanics; Manufacturer Part Number (none) -> CL10B104KB8NNNC; Supplier (none) -> digikey; Supplier P/N  (none) -> 1271276-1000-1-ND; Unit Cost (none) -> 0.15; Weblink (none) -> https://www.digikey.ca/en/products/detail/samsung-electro-m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
- C7: value 100nF -> 4.7uF; Manufacturer (none) -> Samsung Electro-Mechanics; Manufacturer Part Number (none) -> CL10A475KP8NNNC; Supplier (none) -> digikey; Supplier P/N  (none) -> 1276-1044-1-ND; Unit Cost (none) -> 0.15; Weblink (none) -> https://www.digikey.ca/en/products/detail/samsung-electro-m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
- C9: value 22uF -> 4.7uF; footprint Capacitor_SMD:C_0805_2012Metric_Pad1.18x1.45mm_HandSolder -> Capacitor_SMD:C_0603_1608Metric_Pad1.08x0.95mm_HandSolder; Manufacturer (none) -> Samsung Electro-Mechanics; Manufacturer Part Number (none) -> CL10B104KB8NNNC; Supplier (none) -> digikey; Supplier P/N  (none) -> 1271276-1000-1-ND; Unit Cost (none) -> 0.15; Weblink (none) -> https://www.digikey.ca/en/products/detail/samsung-electro-m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
- ESD1: footprint Package_TO_SOT_SMD:SOT-23-3 -> Package_TO_SOT_SMD:SOT-23_Handsoldering; Manufacturer (none) -> SMC Diode Solutions; Manufacturer Part Number (none) -> SM712; Supplier (none) -> digikey; Supplier P/N  (none) -> 1655-SM712CT-ND; Unit Cost (none) -> 0.15; Weblink (none) -> https://www.digikey.ca/en/products/detail/smc-diode-solutio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
- J2: renamed from J1; footprint Connector_PinHeader_1.27mm:PinHeader_1x05_P1.27mm_Horizontal -> Connector_PinHeader_2.54mm:PinHeader_1x05_P2.54mm_Vertical; Manufacturer (none) -> Molex; Manufacturer Part Number (none) -> 0705530109; Supplier (none) -> digikey; Supplier P/N  (none) -> WM4156-ND; Unit Cost (none) -> 3.08; Weblink (none) -> https://www.digikey.ca/en/products/detail/molex/0705530109/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
- LSE1: value JTX310 - Jauch -> ECS-.327-12.5-16-TR3; footprint Crystal:Crystal_SMD_3215-2Pin_3.2x1.5mm -> Crystal:Crystal_SMD_MicroCrystal_CM9V-T1A-2Pin_1.6x1.0mm_HandSoldering; Manufacturer (none) -> Jauch Quartz; Manufacturer Part Number (none) -> Q 0,032768-JTX310-12,5-20-T1-HMR-LF; Supplier (none) -> digikey; Supplier P/N  (none) -> 1908-1341-1-ND; Unit Cost (none) -> 0.7; Weblink (none) -> https://www.digikey.ca/en/products/detail/jauch-quartz/Q-0-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
- R1: value 36k -> 10k; footprint Resistor_SMD:R_0402_1005Metric_Pad0.72x0.64mm_HandSolder -> Resistor_SMD:R_0603_1608Metric_Pad0.98x0.95mm_HandSolder; Manufacturer (none) -> Stackpole Electronics Inc; Manufacturer Part Number (none) -> RMCF0603FT10K0; Supplier (none) -> digikey; Supplier P/N  (none) -> RMCF0603FT10K0CT-ND; Unit Cost (none) -> 0.16; Weblink (none) -> https://www.digikey.ca/en/products/detail/stackpole-electro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
- R2, R7: value 0 -> 10k; footprint Jumper:SolderJumper-2_P1.3mm_Open_TrianglePad1.0x1.5mm -> Resistor_SMD:R_0603_1608Metric_Pad0.98x0.95mm_HandSolder; Manufacturer (none) -> Stackpole Electronics Inc; Manufacturer Part Number (none) -> RMCF0603FT10K0; Supplier (none) -> digikey; Supplier P/N  (none) -> RMCF0603FT10K0CT-ND; Unit Cost (none) -> 0.16; Weblink (none) -> https://www.digikey.ca/en/products/detail/stackpole-electro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
- R25: value 0 -> 50; Manufacturer (none) -> Stackpole Electronics Inc; Manufacturer Part Number (none) -> RMCF0603FT10R0; Supplier (none) -> digikey; Supplier P/N  (none) -> RMCF0603FT10R0CT-ND; Unit Cost (none) -> 0.15; Weblink (none) -> https://www.digikey.ca/en/products/detail/stackpole-electro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
- R3, R4: value 120k -> 10; Manufacturer (none) -> Stackpole Electronics Inc; Manufacturer Part Number (none) -> RMCF0603FT10R0; Supplier (none) -> digikey; Supplier P/N  (none) -> RMCF0603FT10R0CT-ND; Unit Cost (none) -> 0.15; Weblink (none) -> https://www.digikey.ca/en/products/detail/stackpole-electro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
- R5: value 1k -> 10k; footprint Resistor_SMD:R_0402_1005Metric_Pad0.72x0.64mm_HandSolder -> Resistor_SMD:R_0603_1608Metric_Pad0.98x0.95mm_HandSolder; Manufacturer (none) -> Stackpole Electronics Inc; Manufacturer Part Number (none) -> RMCF0603FT10K0; Supplier (none) -> digikey; Supplier P/N  (none) -> RMCF0603FT10K0CT-ND; Unit Cost (none) -> 0.16; Weblink (none) -> https://www.digikey.ca/en/products/detail/stackpole-electro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
- R8: value 120k -> 10k; Manufacturer (none) -> Stackpole Electronics Inc; Manufacturer Part Number (none) -> RMCF0603FT10K0; Supplier (none) -> digikey; Supplier P/N  (none) -> RMCF0603FT10K0CT-ND; Unit Cost (none) -> 0.16; Weblink (none) -> https://www.digikey.ca/en/products/detail/stackpole-electro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
- S1: Manufacturer (none) -> C&K; Manufacturer Part Number (none) -> PTS526 SK15 SMTR2 LFS; Supplier (none) -> digikey; Supplier P/N  (none) -> CKN12221-1-ND; Unit Cost (none) -> 0.22; Weblink (none) -> https://www.digikey.ca/en/products/detail/c-k/PTS526-SK15-S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
- SW1: footprint Button_Switch_SMD:SW_DIP_SPSTx04_Slide_6.7x11.72mm_W8.61mm_P2.54mm_LowProfile -> Button_Switch_SMD:SW_DIP_SPSTx04_Slide_KingTek_DSHP04TS_W7.62mm_P1.27mm
- U3: renamed from U4; value STM32G071CBTx -> STM32G071CBT6; Manufacturer (none) -> STMicroelectronics; Manufacturer Part Number (none) -> STM32G071CBT6; Supplier (none) -> digikey; Supplier P/N  (none) -> 497-18342-ND; Unit Cost (none) -> 6.59; Weblink (none) -> https://www.digikey.ca/en/products/detail/stmicroelectronic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
Connections:
- net EN is gone; now on net GND: R8.2
- net VREF+ is gone; now on net +3V3: U3.5 (VREF+)
- net Vin is gone; now on net CFG3: R7.1
- net +3V3: now also C10.1, C4.1, C5.1, C6.1, C9.1, J2.5 (Pin_5), J3.2 (Pin_2), J4.2 (Pin_2), U1.8 (VCC), U2.1 (VCC), U4.1 (VCC); no longer J2.4 (Pin_4)
- net CFG1: now also R5.1, SW1.5, U3.47 (PB8); no longer SW1.8
- net CFG2: now also SW1.6, U3.46 (PB7), R6.1; no longer SW1.7
- net CFG3: now also SW1.7, U3.45 (PB6); no longer SW1.6
- net CFG4: now also R8.1, SW1.8, U3.44 (PB5); no longer SW1.5
- net CFG_PWR: now also U3.48 (PB9)
- net GND: now also C6.2, R1.2, R5.2, R7.2, C2.2, J3.5 (Pin_5), J4.5 (Pin_5), R6.2, U1.5 (GND), U1.9 (EPAD), U2.3 (GND), U4.3 (GND); no longer R1.1, R25.2, R4.2
- net HEAT: now also U3.39 (PD1); no longer R5.2
- net LPUART_DE: now also R1.1, U3.15 (PA4), U1.2 (*RE), U1.3 (DE); no longer U3.20 (PB1)
- net LP_RxD: now also R2.2, TP4.1, U1.1 (R)
- net LP_TxD: now also TP3.1, U1.4 (D)
- net LSE_OUT: now also C3.1, TP1.1; no longer C4.1
- net NRST: now also J2.4 (Pin_4), C2.1; no longer J2.5 (Pin_5)
- net OUT_A: now also R25.1, R3.1, J1.2 (Pin_2)
- net OUT_B: now also R25.2, R4.1, J1.1 (Pin_1)
- net TEMP: now also U3.22 (PB10)
- net ENC_I_AZM: now reaches U3.11 (PA0)
- net ENC_I_AZM: now also J3.4 (Pin_4)
- net ENC_A_AZM: now reaches U3.12 (PA1)
- net ENC_A_AZM: now also J3.3 (Pin_3)
- net ENC_B_AZM: now reaches U3.17 (PA6)
- net ENC_B_AZM: now also J3.1 (Pin_1)
- net ENC_B_ALT: now reaches U3.18 (PA7)
- net ENC_B_ALT: now also J4.1 (Pin_1)
- net ENC_A_ALT: now reaches U3.19 (PB0)
- net ENC_A_ALT: now also J4.3 (Pin_3)
- net STEP_PWM: now reaches U3.21 (PB2)
- net STEP_DIR: now reaches U3.23 (PB11)
- net STEP_nSLEEP: now reaches U3.24 (PB12)
- net BDC_nSLEEP: now reaches U3.25 (PB13)
- net BDC_DIR: now reaches U3.26 (PB14)
- net ENC_I_ALT: now reaches U3.27 (PB15)
- net ENC_I_ALT: now also J4.4 (Pin_4)
- net END_AZM: now reaches U3.33 (PA11/PA9)
- net END_AZM: now also U2.2 (OUT)
- net MOFF: now reaches U3.40 (PD2)
- net at R3.2: now also U1.6 (A)
- net CLK-PROBE renamed BDC_PWM
- net UART1_RxD renamed END_ALT
- net END_ALT: now also U4.2 (OUT)
- net UART1_TxD: no longer names the net of U3.29 (PA9/UCPD1_DBCC1)
- removed net VCC: R3.1, R8.1
- new net: R4.2, U1.7 (B)
- new net STEP_FAULT: U3.20 (PB1)
- no-connect marks 5 -> 13
Other:
- added sheet POWER & MOTORS (POWER.kicad_sch)
- note added: "ADC_IN11"
- note added: "Configure as internal pull-up"
- note added: "LPTIM1_OUT"
- note added: "LPTIM2_OUT"
- note added: "LPUART1"
- note added: "Push-Pull"
- note added: "R1,R4 - 10 Ohm pulse-proof thickfilm resistors w low error"
- note removed: "/\ CONFIG"
- note removed: "<- COMMUNICATION"
- note removed: "<- POSITIONING"
- note removed: "ESSENTIALS ->"
- note removed: "High quality ceramic cap. must be used for BST pin"
- note removed: "LDO used for filtering"
- note removed: "POWER ->"
- note removed: "R6,R7 - 10 Ohm pulse-proof thickfilm resistors w low error"
- note removed: "Suggested inductor: BOURNS - SRN6045TA-6R3M"
- note removed: "UVLO = 9.5V Vstart = 10V"
- moved on the sheet: C1, J2, LSE1, U3

Commit message: Add files via upload
Other:
- note added: "- All connection pads and header pins should be replaced with JST connectors for assembly convenience and reliability."
- note added: "- Encoder input pins on the MCU are selected incorrectly. Either rewire the encoders accordingly, or fix the circuit and reroute the pins. Consult STM32CubeIDE's setup GUI to configurate proper pinout."
- note added: "- Hall effect latches are used, which means the HIGH signal holds until the sensor senses a source of magnetic flux with the opposite direction. Find a "switch" instead (Texas Instruments have those too)."
- note added: "- The encoders are open-drain output and the MCU's internal pull-up resistors might be too large for higher speeds, add external circuitry to accomodate this if needed."
- note added: "Post-debugging notes:"
- moved on the sheet: C1, C10, C2, C3, C4, C5, C6, C7, C8, C9, ESD1, J1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
