File: POWER.kicad_sch (KiCad schematic)
At the start: 49 parts, among them J3 Conn_01x02, Q1 2N7002LT3G, Q3 2N7002LT3G, Q7 2N7002LT3G, Q8 2N7002LT3G, U2 TPS62933, U3 TMP300, U6 DRV8428, U8 DRV8220DSGR-8p

Commit message: Add files via upload
Parts:
- R13: renamed from R6; value Heater -> Heating trace
- renumbered C21 to C11, C23 to C12, C18 to C13, C4 to C14, C9 to C15, C8 to C16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
Other:
- note added: "POWER & MOTOR DRIVERS"
- note removed: "POWER & MOTOR DRIVING"
- moved on the sheet: C11, C12, C18, C19, H1, H2, H3, H4, H5, H6, JP3, JP4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
